Commit message: Finished model

File: urdf/nugv_core.xacro (robot description, xacro)
@@ -1,4 +1,5 @@
 <?xml version="1.0"?>
 <robot xmlns:xacro="http://www.ros.org/wiki/xacro"  name="nugv_core">
+    <!-- ############################################################################################### -->
     <!-- COLOR -->
     <material name="white">
@@ -14,6 +15,18 @@
         <color rgba="0 0 0 1"/>
     </material>
+    <!-- ############################################################################################### -->
+    <!-- NUGV PROPERTIES -->
+    <!-- Unit: Meters -->
+    <!-- Chasis -->
+    <xacro:property name="chasis_length" value="0.5" />
+    <xacro:property name="chasis_width" value="0.42" />
+    <xacro:property name="chasis_height" value="0.38" />
+    <!-- Thruster -->
+    <xacro:property name="thruster_radius" value="0.05" />
+    <xacro:property name="thruster_length" value="0.05" />
+    <!-- ############################################################################################### -->
     <!-- BASE LINK -->
     <link name="base_link"/>
+    <!-- ############################################################################################### -->
     <!-- CHASSIS LINK -->
     <joint name="chassis_joint" type="fixed">
@@ -24,61 +37,115 @@
         <visual>
             <geometry>
-                        <!-- x    y   z   in meters-->
-                <box size="0.5 0.42 0.38"/>
+                        <!--       x                y               z           in meters-->
+                <box size="${chasis_length} ${chasis_width} ${chasis_height}"/>
+            </geometry>
+            <material name="orange"/>
+        </visual>
+    </link>
+    <!-- ############################################################################################### -->
+    <!-- FRONT LEFT THRUSTER LINK -->
+    <joint name="thruster_front_left_joint" type="continuous">
+        <parent link="base_link"/>
+        <child link="thruster_front_left"/>
+        <origin xyz="0.25 0.21 0" rpy="-${pi/2} 0 ${pi/4}" />
+        <!-- axis of rotation; in this case, thruster rotates around the Z axis -->
+        <axis xyz="0 0 1"/>
+    </joint>
+    <link name="thruster_front_left">
+        <visual>
+            <geometry>
+                <cylinder radius="${thruster_radius}" length="${thruster_length}"/>
             </geometry>
             <material name="white"/>
         </visual>
     </link>
-    <!-- FRONT LEFT THRUSTER LINK -->
-    <joint name="thruster_front_left_joint" type="continuous">
-        <parent link="base_link"/>
-        <child link="thruster_front_left"/>
-        <origin xyz="0.25 0.21 0" rpy="-${pi/2} 0 0" />
-        <axis xyz="0 0 1"/>
-    </joint>
-    <link name="thruster_front_left">
-    </link>
+    <!-- ############################################################################################### -->
     <!-- FRONT RIGHT THRUSTER LINK -->
     <joint name="thruster_front_right_joint" type="continuous">
         <parent link="base_link"/>
         <child link="thruster_front_right"/>
-        <origin xyz="0.25 0.21 0" rpy="-${pi/2} 0 0" />
+        <origin xyz="0.25 -0.21 0" rpy="-${pi/2} 0 -${pi/4}" />
+        <!-- axis of rotation; in this case, thruster rotates around the Z axis -->
         <axis xyz="0 0 1"/>
     </joint>
     <link name="thruster_front_right">
+        <visual>
+            <geometry>
+                <cylinder radius="${thruster_radius}" length="${thruster_length}"/>
+            </geometry>
+            <material name="white"/>
+        </visual>
     </link>
+    <!-- ############################################################################################### -->
     <!-- BACK LEFT THRUSTER LINK -->
     <joint name="thruster_back_left_joint" type="continuous">
         <parent link="base_link"/>
         <child link="thruster_back_left"/>
-        <origin xyz="0.25 0.21 0" rpy="-${pi/2} 0 0" />
+        <origin xyz="-0.25 0.21 0" rpy="-${pi/2} 0 -${pi/4}" />
+        <!-- axis of rotation; in this case, thruster rotates around the Z axis -->
         <axis xyz="0 0 1"/>
     </joint>
     <link name="thruster_back_left">
+        <visual>
+            <geometry>
+                <cylinder radius="${thruster_radius}" length="${thruster_length}"/>
+            </geometry>
+            <material name="white"/>
+        </visual>
     </link>
+    <!-- ############################################################################################### -->
     <!-- BACK RIGHT THRUSTER LINK -->
     <joint name="thruster_back_right_joint" type="continuous">
         <parent link="base_link"/>
         <child link="thruster_back_right"/>
-        <origin xyz="0.25 0.21 0" rpy="-${pi/2} 0 0" />
+        <origin xyz="-0.25 -0.21 0" rpy="-${pi/2} 0 ${pi/4}" />
+        <!-- axis of rotation; in this case, thruster rotates around the Z axis -->
         <axis xyz="0 0 1"/>
     </joint>
     <link name="thruster_back_right">
+        <visual>
+            <geometry>
+                <cylinder radius="${thruster_radius}" length="${thruster_length}"/>
+            </geometry>
+            <material name="white"/>
+        </visual>
     </link>
+    <!-- ############################################################################################### -->
     <!-- FRONT DEPTH THRUSTER LINK -->
     <joint name="depth_thruster_front" type="continuous">
         <parent link="base_link"/>
         <child link="depth_thruster_front"/>
+        <origin xyz="0.25 0 0" rpy="${pi} 0 0" />
+        <!-- axis of rotation; in this case, thruster rotates around the Z axis -->
+        <axis xyz="0 0 1"/>
     </joint>
     <link name="depth_thruster_front">
+        <visual>
+            <geometry>
+                <cylinder radius="${thruster_radius}" length="${thruster_length}"/>
+            </geometry>
+            <material name="blue"/>
+        </visual>
     </link>
+    <!-- ############################################################################################### -->
     <!-- BACK DEPTH THRUSTER LINK -->
     <joint name="depth_thruster_back" type="continuous">
         <parent link="base_link"/>
         <child link="depth_thruster_back"/>
+        <origin xyz="-0.25 0 0" rpy="${pi} 0 0" />
+        <!-- axis of rotation; in this case, thruster rotates around the Z axis -->
+        <axis xyz="0 0 1"/>
     </joint>
     <link name="depth_thruster_back">
+        <visual>
+            <geometry>
+                <cylinder radius="${thruster_radius}" length="${thruster_length}"/>
+            </geometry>
+            <material name="blue"/>
+        </visual>
     </link>
+    <!-- ############################################################################################### -->
     <!-- IMU LINK -->
+    <!-- ############################################################################################### -->
     <!-- DIGITAL CAMERA LINK -->
 </robot>

Commit message: Fixed orientation

File: urdf/nugv_core.xacro (robot description, xacro)
@@ -65,5 +65,5 @@
         <parent link="base_link"/>
         <child link="thruster_front_right"/>
-        <origin xyz="0.25 -0.21 0" rpy="-${pi/2} 0 -${pi/4}" />
+        <origin xyz="0.25 -0.21 0" rpy="-${pi/2} 0 ${pi*3/4}" />
         <!-- axis of rotation; in this case, thruster rotates around the Z axis -->
         <axis xyz="0 0 1"/>
@@ -82,5 +82,5 @@
         <parent link="base_link"/>
         <child link="thruster_back_left"/>
-        <origin xyz="-0.25 0.21 0" rpy="-${pi/2} 0 -${pi/4}" />
+        <origin xyz="-0.25 0.21 0" rpy="-${pi/2} 0 ${pi*3/4}" />
         <!-- axis of rotation; in this case, thruster rotates around the Z axis -->
         <axis xyz="0 0 1"/>

Commit message: Added imu frame

File: urdf/nugv_core.xacro (robot description, xacro)
@@ -113,5 +113,5 @@
     <!-- ############################################################################################### -->
     <!-- FRONT DEPTH THRUSTER LINK -->
-    <joint name="depth_thruster_front" type="continuous">
+    <joint name="depth_thruster_front_joint" type="continuous">
         <parent link="base_link"/>
         <child link="depth_thruster_front"/>
@@ -130,5 +130,5 @@
     <!-- ############################################################################################### -->
     <!-- BACK DEPTH THRUSTER LINK -->
-    <joint name="depth_thruster_back" type="continuous">
+    <joint name="depth_thruster_back_joint" type="continuous">
         <parent link="base_link"/>
         <child link="depth_thruster_back"/>
@@ -147,4 +147,17 @@
     <!-- ############################################################################################### -->
     <!-- IMU LINK -->
+    <joint name="imu_joint" type="continuous">
+        <parent link="base_link"/>
+        <child link="imu"/>
+        <origin xyz="0 0 0.1" rpy="0 0 0" />
+    </joint>
+    <link name="imu">
+        <visual>
+            <geometry>
+                <cylinder radius="0.05" length="0.01"/>
+            </geometry>
+            <material name="black"/>
+        </visual>
+    </link>
     <!-- ############################################################################################### -->
     <!-- DIGITAL CAMERA LINK -->

Commit message: Small update

File: urdf/nugv_core.xacro (robot description, xacro)
@@ -1,5 +1,5 @@
 <?xml version="1.0"?>
 <robot xmlns:xacro="http://www.ros.org/wiki/xacro"  name="nugv_core">
-    <!-- ############################################################################################### -->
+    <!-- ********************************************************************************* -->
     <!-- COLOR -->
     <material name="white">
@@ -15,5 +15,5 @@
         <color rgba="0 0 0 1"/>
     </material>
-    <!-- ############################################################################################### -->
+    <!-- ********************************************************************************* -->
     <!-- NUGV PROPERTIES -->
     <!-- Unit: Meters -->
@@ -25,8 +25,8 @@
     <xacro:property name="thruster_radius" value="0.05" />
     <xacro:property name="thruster_length" value="0.05" />
-    <!-- ############################################################################################### -->
+    <!-- ********************************************************************************* -->
     <!-- BASE LINK -->
     <link name="base_link"/>
-    <!-- ############################################################################################### -->
+    <!-- ********************************************************************************* -->
     <!-- CHASSIS LINK -->
     <joint name="chassis_joint" type="fixed">
@@ -43,5 +43,5 @@
         </visual>
     </link>
-    <!-- ############################################################################################### -->
+    <!-- ********************************************************************************* -->
     <!-- FRONT LEFT THRUSTER LINK -->
     <joint name="thruster_front_left_joint" type="continuous">
@@ -60,5 +60,5 @@
         </visual>
     </link>
-    <!-- ############################################################################################### -->
+    <!-- ********************************************************************************* -->
     <!-- FRONT RIGHT THRUSTER LINK -->
     <joint name="thruster_front_right_joint" type="continuous">
@@ -77,5 +77,5 @@
         </visual>
     </link>
-    <!-- ############################################################################################### -->
+    <!-- ********************************************************************************* -->
     <!-- BACK LEFT THRUSTER LINK -->
     <joint name="thruster_back_left_joint" type="continuous">
@@ -94,5 +94,5 @@
         </visual>
     </link>
-    <!-- ############################################################################################### -->
+    <!-- ********************************************************************************* -->
     <!-- BACK RIGHT THRUSTER LINK -->
     <joint name="thruster_back_right_joint" type="continuous">
@@ -111,5 +111,5 @@
         </visual>
     </link>
-    <!-- ############################################################################################### -->
+    <!-- ********************************************************************************* -->
     <!-- FRONT DEPTH THRUSTER LINK -->
     <joint name="depth_thruster_front_joint" type="continuous">
@@ -128,5 +128,5 @@
         </visual>
     </link>
-    <!-- ############################################################################################### -->
+    <!-- ********************************************************************************* -->
     <!-- BACK DEPTH THRUSTER LINK -->
     <joint name="depth_thruster_back_joint" type="continuous">
@@ -145,7 +145,7 @@
         </visual>
     </link>
-    <!-- ############################################################################################### -->
+    <!-- ********************************************************************************* -->
     <!-- IMU LINK -->
-    <joint name="imu_joint" type="continuous">
+    <joint name="imu_joint" type="fixed">
         <parent link="base_link"/>
         <child link="imu"/>
@@ -160,5 +160,7 @@
         </visual>
     </link>
-    <!-- ############################################################################################### -->
+    <!-- ********************************************************************************* -->
+    <!-- SONAR LINK -->
+    <!-- ********************************************************************************* -->
     <!-- DIGITAL CAMERA LINK -->
 </robot>

Commit message: Added sonar frame

File: urdf/nugv_core.xacro (robot description, xacro)
@@ -162,4 +162,17 @@
     <!-- ********************************************************************************* -->
     <!-- SONAR LINK -->
+    <joint name="sonar_joint" type="fixed">
+        <parent link="base_link"/>
+        <child link="sonar"/>
+        <origin xyz="0.25 -0.21 ${chasis_height/2}" rpy="0 0 0" />
+    </joint>
+    <link name="sonar">
+        <visual>
+            <geometry>
+                <cylinder radius="0.05" length="0.05"/>
+            </geometry>
+            <material name="blue"/>
+        </visual>
+    </link>
     <!-- ********************************************************************************* -->
     <!-- DIGITAL CAMERA LINK -->
